File: TXB0108/TXB0108.kicad_pcb (KiCad board)
At the start: 2 copper layers, 15.2 x 25.4 mm, 10 parts, among them J1 Conn_01x10, J2 Conn_01x10

Commit message: SOIC8 Changed to TSSOP8
Other:
- board text added: "VA : 1.2V - 3.6V VB : 1.7V - 5.5V"
- board text removed: "LV : 1.2V - 3.6V HV : 1.7V - 5.5V"
Changed lines of the file:
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@@
     (34 B.Paste user hide)
     (35 F.Paste user hide)
-    (36 B.SilkS user hide)
+    (36 B.SilkS user)
     (37 F.SilkS user)
     (38 B.Mask user hide)
@@
     )
   )
-  (gr_text "LV : 1.2V - 3.6V\nHV : 1.7V - 5.5V" (at 137.541 115.57 270) (layer B.SilkS)
+  (gr_text "VA : 1.2V - 3.6V\nVB : 1.7V - 5.5V" (at 137.541 115.57 270) (layer B.SilkS)
     (effects (font (size 1 1) (thickness 0.15)) (justify mirror))
   )

Commit message: Final Revisions
Routing:
- net /VccB: track 4.92 -> 12.3 mm, vias 0 -> 1
Changed lines of the file:
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@@
     (thickness 1.6)
     (drawings 17)
-    (tracks 81)
+    (tracks 84)
     (zones 0)
     (modules 10)
@@
   (segment (start 140.081 112.971) (end 140.081 111.68888) (width 0.25) (layer F.Cu) (net 3))
   (segment (start 140.081 111.68888) (end 140.081 111.633) (width 0.25) (layer F.Cu) (net 3))
+  (via (at 141.478 110.118) (size 0.8) (drill 0.4) (layers F.Cu B.Cu) (net 3))
+  (segment (start 141.478 107.442) (end 144.78 104.14) (width 0.25) (layer B.Cu) (net 3))
+  (segment (start 141.478 110.118) (end 141.478 107.442) (width 0.25) (layer B.Cu) (net 3))
   (segment (start 136.455 115.895) (end 135.48 115.895) (width 0.25) (layer F.Cu) (net 4))
   (segment (start 136.97712 116.41712) (end 136.455 115.895) (width 0.25) (layer F.Cu) (net 4))

Commit message: Silkscreen Edits
Dimensions moved to Drawings Layer
Other:
- rule pad_to_mask_clearance: 0.051 -> 0
- rule solder_mask_min_width: 0.25 -> 0.1
Changed lines of the file:
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@@
     (pad_size 1.7 1.7)
     (pad_drill 1)
-    (pad_to_mask_clearance 0.051)
-    (solder_mask_min_width 0.25)
+    (pad_to_mask_clearance 0)
+    (solder_mask_min_width 0.1)
     (aux_axis_origin 0 0)
     (visible_elements 7FFFFFFF)
     (pcbplotparams
-      (layerselection 0x010fc_ffffffff)
+      (layerselection 0x010f0_ffffffff)
       (usegerberextensions false)
       (usegerberattributes false)
@@
       (viasonmask false)
       (mode 1)
-      (useauxorigin false)
+      (useauxorigin true)
       (hpglpennumber 1)
       (hpglpenspeed 20)
@@
       (psa4output false)
       (plotreference true)
-      (plotvalue true)
+      (plotvalue false)
       (plotinvisibletext false)
       (padsonsilk false)
@@
       (outputformat 1)
       (mirror false)
-      (drillshape 1)
+      (drillshape 0)
       (scaleselection 1)
-      (outputdirectory ""))
+      (outputdirectory "../../Gerbers/TXB0108/"))
   )
   (net 0 "")
@@
     )
   )
-  (dimension 22.86 (width 0.12) (layer F.SilkS)
-    (gr_text "22.860 mm" (at 149.86 115.57 270) (layer F.SilkS)
+  (dimension 22.86 (width 0.12) (layer Dwgs.User)
+    (gr_text "22.860 mm" (at 149.86 115.57 270) (layer Dwgs.User)
       (effects (font (size 1 1) (thickness 0.15)) hide)
     )
@@
     (arrow2b (pts (xy 148.59 104.14) (xy 149.176421 105.266504)))
   )
-  (dimension 25.4 (width 0.12) (layer F.SilkS)
-    (gr_text "25.400 mm" (at 152.654 115.57 270) (layer F.SilkS)
+  (dimension 25.4 (width 0.12) (layer Dwgs.User)
+    (gr_text "25.400 mm" (at 152.654 115.57 270) (layer Dwgs.User)
       (effects (font (size 1 1) (thickness 0.15)) hide)
     )
@@
     (arrow2b (pts (xy 151.384 102.87) (xy 151.970421 103.996504)))
   )
-  (dimension 12.7 (width 0.12) (layer F.SilkS)
-    (gr_text "12.700 mm" (at 138.43 99.822) (layer F.SilkS)
+  (dimension 12.7 (width 0.12) (layer Dwgs.User)
+    (gr_text "12.700 mm" (at 138.43 99.822) (layer Dwgs.User)
       (effects (font (size 1 1) (thickness 0.15)) hide)
     )
@@
     (arrow2b (pts (xy 132.08 101.092) (xy 133.206504 100.505579)))
   )
-  (dimension 15.24 (width 0.12) (layer F.SilkS)
-    (gr_text "15.240 mm" (at 138.43 97.409) (layer F.SilkS)
+  (dimension 15.24 (width 0.12) (layer Dwgs.User)
+    (gr_text "15.240 mm" (at 138.43 97.409) (layer Dwgs.User)
       (effects (font (size 1 1) (thickness 0.15)) hide)
     )

Commit message: Part Numbers Added
Parts:
- moved C2 104.3 mm to (70.5, 32.6)
- moved G*** 104.3 mm to (67.4, 39.1)
- moved J1 104.3 mm to (61.1, 27.7)
- moved J2 104.3 mm to (73.8, 27.7)
- moved R1 104.3 mm to (67.4, 33.7)
- moved REF** 104.3 mm to (67.4, 48.6)
- moved REF** 104.3 mm to (67.4, 29.6)
- moved TXB0108 104.3 mm to (67.4, 39.1)
- moved C1 104.3 mm to (64.5, 32.6)
- moved G*** 104.3 mm to (67.4, 44.4)
